File: circuit/zeabus_hydrophone.kicad_pcb (KiCad board)
At the start: 4 copper layers, 100 x 70 mm, 157 parts, among them CN1 EPS.00.250.NTN, CN2 EPS.00.250.NTN, CN3 EPS.00.250.NTN, CN4 EPS.00.250.NTN, CON1 ZTEX-V2-FPGA, J1 JTAG, U1 AD9248, U10 MAX5387LAUD+T (10k), U11 MAX5387LAUD+T (10k), U2 AD9248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

Commit message: Finish PCB routing. Some device drivers in firmware are tested
Parts:
- moved R51 39.0 mm to (116.2, 60.4), turned to 270 degrees
- moved R52 38.9 mm to (113.6, 60.4), turned to 270 degrees
- moved C65 3.35 mm to (143.3, 75.8), turned to 270 degrees
- moved C67 3.35 mm to (143.3, 72.5), turned to 270 degrees
- moved R40 1.53 mm to (145.8, 74.9)
- moved R48 1.50 mm to (145.8, 73.4)
- moved RN1 1.20 mm to (118.0, 110.0)
- moved RN2 1.20 mm to (118.0, 106.3)
- moved RN5 0.68 mm to (118.5, 78.8)
- moved RN6 0.65 mm to (118.6, 75.1)
- moved C70 0.42 mm to (162.3, 64.2)
- moved C60 0.20 mm to (162.3, 97.8)
- moved C34 0.18 mm to (136.4, 84.0)
- moved C35 0.18 mm to (134.9, 84.0)
- moved C37 0.18 mm to (136.4, 80.7)
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Connections:
- CON1 pad A29: /SDA -> Net-(CON1-PadA29)
- CON1 pad A30: /SCL -> Net-(CON1-PadA30)
- CON1 pad D14: Net-(CON1-PadD14) -> /SDA
- CON1 pad D15: Net-(CON1-PadD15) -> /SCL
Routing:
- net VDD: track 0.00 -> 178.7 mm, vias 0 -> 16
- net GNDA: track 0.00 -> 153.0 mm, vias 0 -> 67
- net /SDA: track 0.00 -> 122.8 mm, vias 0 -> 5
- net VBUS: track 0.00 -> 119.2 mm
- net Net-(CON1-PadC31): track 0.00 -> 119.0 mm, vias 0 -> 1
- net /SCL: track 0.00 -> 117.0 mm, vias 0 -> 3
- net Net-(CON1-PadD31): track 0.00 -> 111.4 mm, vias 0 -> 1
- net Net-(CON1-PadA31): track 0.00 -> 89.1 mm, vias 0 -> 1
- net Net-(CON1-PadA32): track 0.00 -> 83.8 mm, vias 0 -> 1
- net Net-(CON1-PadB31): track 0.00 -> 83.4 mm, vias 0 -> 1
- net VDDA: track 0.00 -> 63.2 mm, vias 0 -> 17
- net /RESn: track 0.00 -> 53.6 mm
- net /analog/VR4_L: track 0.00 -> 39.9 mm, vias 0 -> 2
- net /analog/VR2_L: track 0.00 -> 38.9 mm, vias 0 -> 2
- net Net-(CON1-PadC3): track 0.00 -> 37.2 mm
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Other:
- net class Default: clearance 0.2 -> 0.15
- net class VBUS added: clearance 0.2, trace_width 0.5, via_dia 0.45, via_drill 0.2
- rule trace_clearance: 0.2 -> 0.15
- board text added: "Zeabus Hydrophone by Akrapong Patchararungruang V.3.0.1"
